Commit message: multi kownbot corepration

File: kownbot_description/urdf/include/common_sensors.xacro (robot description, xacro)
@@ -85,6 +85,6 @@
       <!-- plugin_name is either libgazebo_ros_laser.so or libgazebo_ros_gpu_laser.so-->
       <plugin name="gazebo_ros_head_hokuyo_controller" filename="${plugin_name}">
-        <topicName>/diffbot/scan</topicName>
-        <frameName>${prefix}_laser_link</frameName>
+        <topicName>/$(arg kbot_name)/scan</topicName>
+        <frameName>$(arg kbot_name)/${prefix}_laser_link</frameName>
       </plugin>
     </sensor>
@@ -161,5 +161,5 @@
         <alwaysOn>true</alwaysOn>
         <updateRate>0.0</updateRate>
-        <cameraName>diffbot/camera1</cameraName>
+        <cameraName>$(arg kbot_name)/camera1</cameraName>
         <imageTopicName>image_raw</imageTopicName>
         <cameraInfoTopicName>camera_info</cameraInfoTopicName>

File: kownbot_description/urdf/include/robot.gazebo.xacro (robot description, xacro)
@@ -2,9 +2,9 @@
 <robot xmlns:xacro="http://ros.org/wiki/xacro">
   <!-- ros_control plugin -->
-  <xacro:macro name="gazebo_ros_control" params="robotNamespace robotSimType:=gazebo_ros_control/DefaultRobotHWSim">
+  <xacro:macro name="gazebo_ros_control" params="robotSimType:=gazebo_ros_control/DefaultRobotHWSim">
     <gazebo>
       <plugin name="gazebo_ros_control" filename="libgazebo_ros_control.so">
-        <robotNamespace>${robotNamespace}</robotNamespace>
-        <!--robotParam>/robot_description</robotParam-->
+        <robotNamespace>$(arg kbot_name)</robotNamespace>
+        <robotParam>$(arg kbot_name)/robot_description</robotParam>
         <robotSimType>${robotSimType}</robotSimType>
       </plugin>

File: kownbot_description/urdf/kownbot.urdf.xacro (robot description, xacro)
@@ -34,5 +34,6 @@
   <xacro:wheel prefix="front_left" reflect="1"
                       wheel_props="${front_wheel_props}"
-                      base_props="${base_props}" >
+                      base_props="${base_props}"
+                       >
   </xacro:wheel>
   <!-- Motors -->
@@ -48,8 +49,9 @@
   <xacro:laser prefix="rplidar" parent_link="base_link"
                    sensor_prop="${sensor_prop}"
-                   enable_gpu="${sensor_prop['laser']['enable_gpu']}">
+                   enable_gpu="${sensor_prop['laser']['enable_gpu']}"
+                   >
   </xacro:laser>
   <!-- Gazebo -->
-  <xacro:gazebo_ros_control robotNamespace="/kownbot">
+  <xacro:gazebo_ros_control >
   </xacro:gazebo_ros_control>
 </robot>
